File: plain60-flex-edition.kicad_pcb (KiCad board)
At the start: 2 copper layers, 284.7 x 94.2 mm, 175 parts, among them J1 HRO-TYPE-C-31-M-12, J2 ISP, J3 ai03_ud, K1 KEYSW, K10 KEYSW, K11 KEYSW, K12 KEYSW, K13 KEYSW, K14 KEYSW, K15 KEYSW, K15-1 KEYSW, K16 KEYSW, K17 KEYSW, K18 KEYSW, K19 KEYSW, K2 KEYSW, K20 KEYSW, K21 KEYSW, K22 KEYSW, K23 KEYSW, K24 KEYSW, K25 KEYSW, K26 KEYSW, K27 KEYSW, K28 KEYSW, K29 KEYSW, K3 KEYSW, K31 KEYSW, K31-1 KEYSW, K32 KEYSW, K33 KEYSW, K34 KEYSW, K35 KEYSW, K36 KEYSW, K37 KEYSW, K38 KEYSW, K39 KEYSW, K4 KEYSW, K40 KEYSW, K41 KEYSW, K42 KEYSW, K43 KEYSW, K44 KEYSW, K44-1 KEYSW, K46 KEYSW, K46-1 KEYSW, K47 KEYSW, K48 KEYSW, K49 KEYSW, K5 KEYSW, K50 KEYSW, K51 KEYSW, K52 KEYSW, K53 KEYSW, K54 KEYSW, K55 KEYSW, K56 KEYSW, K57 KEYSW, K58 KEYSW, K58-1 KEYSW, K59 KEYSW, K6 KEYSW, K61 KEYSW, K61-1 KEYSW, K62 KEYSW, K62-1 KEYSW, K63 KEYSW, K63-1 KEYSW, K67 KEYSW, K67-1 KEYSW, K7 KEYSW, K71 KEYSW, K72 KEYSW, K72-1 KEYSW, K73 KEYSW, K73-1 KEYSW, K74 KEYSW, K74-1 KEYSW, K8 KEYSW, K9 KEYSW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

Commit message: added first iteration of refactoring
Parts:
- removed C1: 1u, Keeb_components:C_0805
- removed C2, C3, C4, C5: 0.1u, Keeb_components:C_0805
- removed C6: 4.7u, Keeb_components:C_0805
- removed F1: Polyfuse, Keeb_components:R_0805
- removed J2: ISP, Keeb_components:isp_standard
- removed J3: ai03_ud, Keeb_components:JST_SH_SM04B-SRSS-TB_1x04-1MP_P1.00mm_Horizontal
- removed K46-1: KEYSW, Keeb_switches:CHERRY_PLATE_125H
- removed LS1: Speaker, Keeb_components:speaker_AST1109MLTRQ
- removed R1, R2: 22, Keeb_components:R_0805
- removed R3, R4: 5.1k, Keeb_components:R_0805
- removed R5, R6: 10k, Keeb_components:R_0805
- removed SW1: SW_PUSH, Button_Switch_SMD:SW_SPST_TL3342
- removed U2: USBLC6-2SC6, Keeb_components:USBLC6-2SC6
- removed X1: XTAL_GND, Keeb_components:Resonator_SMD_muRata_CSTNExxV-3Pin-p1.2
- added ?: , , F.Cu at (75.2, 3.84)
- added ?: , , F.Cu at (77.0, 3.84)
- added ?: , , F.Cu at (73.4, 3.84)
- J1: value HRO-TYPE-C-31-M-12 -> 4P4C; footprint Keeb_components:HRO-TYPE-C-31-M-12 -> Connector_JST:JST_PH_S4B-PH-K_1x04_P2.00mm_Horizontal; moved to F.Cu
- U1: value ATmega32U4 -> ProS3; footprint Keeb_components:ATMEGA32U4 -> footprints2:ProS3_TH; moved to F.Cu
- moved J1 41.4 mm to (59.5, 5.84), turned to 180 degrees
- moved K31 26.2 mm to (42.9, 47.6)
- moved K32 26.2 mm to (16.7, 47.6)
- moved D1 21.4 mm to (15.8, 16.8), turned to 180 degrees
- moved U1 18.0 mm to (28.8, 23.7), turned to 0 degrees
- moved D16 9.80 mm to (7.63, 20.0), turned to -90 degrees
- turned S1 to 180 degrees
Connections:
- D32 pad 2: Net-(D32-Pad2) -> Net-(D31-Pad2)
- J1 pad 2: VBUS -> 5V
- J1 pad 3: (no net) -> display SDA
- J1 pad 4: Net-(J1-Pad4) -> display SCL
- K31 pad 1: Net-(D31-Pad2) -> Net-(D32-Pad2)
- K31 pad 2: col0 -> col1
- K32 pad 1: Net-(D32-Pad2) -> Net-(D31-Pad2)
- K32 pad 2: col1 -> col0
- U1 pad 1: row4 -> unconnected-(U1-Pad1)
- U1 pad 10: MOSI -> col8
- U1 pad 12: Net-(LS1-Pad1) -> col9
- U1 pad 13: RST -> col10
- U1 pad 14: VCC -> col11
- U1 pad 15: GND -> col12
- U1 pad 16: Net-(U1-Pad16) -> col13
- U1 pad 17: Net-(U1-Pad17) -> col14
- U1 pad 18: col2 -> col3
- U1 pad 19: col1 -> col2
- U1 pad 2: VCC -> GND
- U1 pad 20: col0 -> rgb R1
- U1 pad 21: col3 -> row4
- U1 pad 22: col4 -> row3
- U1 pad 23: GND -> rx
- U1 pad 24: VCC -> tx
- U1 pad 25: row3 -> unconnected-(U1-Pad25)
- U1 pad 26: row2 -> unconnected-(U1-Pad26)
- U1 pad 27: row1 -> pin03 unused
- U1 pad 28: row0 -> col1
- U1 pad 29: col5 -> display SDA
- U1 pad 3: Net-(R2-Pad2) -> 5V
- U1 pad 30: col7 -> display SCL
- U1 pad 31: col8 -> col0
- U1 pad 32: col9 -> row2
- U1 pad 33: Net-(R6-Pad2) -> row1
- U1 pad 34: VCC -> row0
- U1 pad 4: Net-(R1-Pad1) -> unconnected-(U1-Pad4)
- U1 pad 5: GND -> unconnected-(U1-Pad5)
- U1 pad 6: Net-(C1-Pad1) -> col4
- U1 pad 7: VCC -> col5
- U1 pad 8: Net-(H1-Pad1) -> col6
- U1 pad 9: SCK -> col7
Routing:
- net GND: track 245.5 -> 48.0 mm, vias 22 -> 3
- net Net-(LS1-Pad1): track 187.3 -> 0.00 mm, vias 2 -> 0
- net VCC: track 136.1 -> 0.00 mm, vias 14 -> 0
- net rgb R1: track 0.00 -> 95.0 mm, vias 0 -> 4
- net RST: track 56.9 -> 0.00 mm, vias 3 -> 0
- net 5V: track 0.00 -> 53.4 mm, vias 0 -> 3
- net row2: track 243.5 -> 289.8 mm, vias 0 -> 1
- net display SDA: track 0.00 -> 45.8 mm, vias 0 -> 1
- net display SCL: track 0.00 -> 41.9 mm, vias 0 -> 3
- net col6: track 547.6 -> 585.8 mm, vias 1 -> 3
- net col5: track 281.1 -> 316.3 mm, vias 1 -> 3
- net VBUS: track 34.1 -> 0.00 mm, vias 5 -> 0
- net col7: track 365.7 -> 398.8 mm, vias 1 -> 3
- net col8: track 346.9 -> 379.2 mm, vias 1 -> 3
- net MOSI: track 29.9 -> 0.00 mm
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- removed copper zone on B.Cu, net GND
- removed copper zone on F.Cu, net GND
Other:
- board text added: "5V"
- board text added: "IO40"
- board text added: "customized by fancy-mech.eu"
- board text removed: "Speaker AST1109MLTRQ Pin B7"

Commit message: tuning
Parts:
- J1, U1: moved to B.Cu
- moved J1 5.98 mm to (53.5, 6.02), turned to 0 degrees
- moved U1 0.25 mm to (28.8, 23.4), turned to 180 degrees
Connections:
- U1 pad 31: col0 -> unconnected-(U1-Pad31)
- U1 pad 5: unconnected-(U1-Pad5) -> col0
Routing:
- net col2: track 156.6 -> 134.4 mm, vias 2 -> 1
- net rgb R1: track 95.0 -> 75.0 mm, vias 4 -> 2
- net col4: track 202.1 -> 218.2 mm
- net display SDA: track 45.8 -> 30.0 mm
- net col3: track 178.1 -> 162.9 mm, vias 2 -> 3
- net 5V: track 53.4 -> 67.9 mm, vias 3 -> 2
- net GND: track 48.0 -> 61.4 mm, vias 3 -> 1
- net row4: track 273.3 -> 283.9 mm
- net display SCL: track 41.9 -> 32.7 mm, vias 3 -> 1
- net row3: track 283.4 -> 292.4 mm
- net row1: track 279.3 -> 285.9 mm
- net col5: track 316.3 -> 322.3 mm
- net col10: track 423.3 -> 417.9 mm
- net col0: track 127.6 -> 123.0 mm
- net Net-(D2-Pad2): track 18.8 -> 14.2 mm
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Other:
- board text removed: "UDB"

Commit message: added underglow leds
Parts:
- removed ? (x3): , 
- added LED1: WS2812B, LED_SMD:LED_WS2812B_PLCC4_5.0x5.0mm_P3.2mm, B.Cu at (7.88, 17.3)
- added LED10: WS2812B, LED_SMD:LED_WS2812B_PLCC4_5.0x5.0mm_P3.2mm, B.Cu at (210.1, 71.7)
- added LED11: WS2812B, LED_SMD:LED_WS2812B_PLCC4_5.0x5.0mm_P3.2mm, B.Cu at (170.2, 71.9)
- added LED12: WS2812B, LED_SMD:LED_WS2812B_PLCC4_5.0x5.0mm_P3.2mm, B.Cu at (129.3, 72.2)
- added LED13: WS2812B, LED_SMD:LED_WS2812B_PLCC4_5.0x5.0mm_P3.2mm, B.Cu at (95.8, 71.9)
- added LED14: WS2812B, LED_SMD:LED_WS2812B_PLCC4_5.0x5.0mm_P3.2mm, B.Cu at (54.9, 72.7)
- added LED15: WS2812B, LED_SMD:LED_WS2812B_PLCC4_5.0x5.0mm_P3.2mm, B.Cu at (17.5, 71.4)
- added LED16: WS2812B, LED_SMD:LED_WS2812B_PLCC4_5.0x5.0mm_P3.2mm, B.Cu at (18.0, 54.6)
- added LED2: WS2812B, LED_SMD:LED_WS2812B_PLCC4_5.0x5.0mm_P3.2mm, B.Cu at (47.5, 14.8)
- added LED3: WS2812B, LED_SMD:LED_WS2812B_PLCC4_5.0x5.0mm_P3.2mm, B.Cu at (87.1, 15.3)
- added LED4: WS2812B, LED_SMD:LED_WS2812B_PLCC4_5.0x5.0mm_P3.2mm, B.Cu at (125.5, 15.3)
- added LED5: WS2812B, LED_SMD:LED_WS2812B_PLCC4_5.0x5.0mm_P3.2mm, B.Cu at (168.7, 14.5)
- added LED6: WS2812B, LED_SMD:LED_WS2812B_PLCC4_5.0x5.0mm_P3.2mm, B.Cu at (216.4, 15.0)
- added LED7: WS2812B, LED_SMD:LED_WS2812B_PLCC4_5.0x5.0mm_P3.2mm, B.Cu at (267.5, 16.0)
- added LED8: WS2812B, LED_SMD:LED_WS2812B_PLCC4_5.0x5.0mm_P3.2mm, B.Cu at (274.8, 44.7)
- added LED9: WS2812B, LED_SMD:LED_WS2812B_PLCC4_5.0x5.0mm_P3.2mm, B.Cu at (263.2, 74.5)
- moved D16 8.42 mm to (4.84, 28.0), turned to 90 degrees
- moved D44 2.35 mm to (272.3, 51.2)
Connections:
- net pin03 unused renamed pin27 unused
- U1 pad 31: unconnected-(U1-Pad31) -> pin31 unused
Routing:
- net GND: track 61.4 -> 708.9 mm, vias 1 -> 12
- net 5V: track 67.9 -> 694.9 mm, vias 2 -> 14
- net Net-(LED10-Pad4): track 0.00 -> 50.0 mm, vias 0 -> 2
- net Net-(LED6-Pad2): track 0.00 -> 49.3 mm, vias 0 -> 2
- net Net-(LED7-Pad2): track 0.00 -> 48.3 mm, vias 0 -> 2
- net Net-(LED5-Pad2): track 0.00 -> 45.5 mm, vias 0 -> 2
- net Net-(LED4-Pad2): track 0.00 -> 42.2 mm, vias 0 -> 2
- net Net-(LED1-Pad2): track 0.00 -> 41.4 mm, vias 0 -> 2
- net Net-(LED13-Pad2): track 0.00 -> 39.3 mm, vias 0 -> 2
- net Net-(LED11-Pad2): track 0.00 -> 39.1 mm, vias 0 -> 2
- net Net-(LED8-Pad2): track 0.00 -> 38.9 mm, vias 0 -> 2
- net Net-(LED14-Pad2): track 0.00 -> 38.6 mm
- net Net-(LED2-Pad2): track 0.00 -> 38.0 mm
- net Net-(LED10-Pad2): track 0.00 -> 38.0 mm, vias 0 -> 2
- net Net-(LED3-Pad2): track 0.00 -> 36.6 mm
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